Commit message: Updated mesh file paths in urdf

File: mani_skill2_real2sim/assets/descriptions/panda_robotiq_85.urdf (robot description, URDF)
Before this commit: robot panda, 21 links, 20 joints
Links:
- link panda_link0: geometry collision mesh filename=franka_description/meshes/collision/link0.stl; visual mesh filename=franka_description/meshes/visual/link0.dae
- link panda_link1: geometry collision mesh filename=franka_description/meshes/collision/link1.stl; visual mesh filename=franka_description/meshes/visual/link1.dae
- link panda_link2: geometry collision mesh filename=franka_description/meshes/collision/link2.stl; visual mesh filename=franka_description/meshes/visual/link2.dae
- link panda_link3: geometry collision mesh filename=franka_description/meshes/collision/link3.stl; visual mesh filename=franka_description/meshes/visual/link3.dae
- link panda_link4: geometry collision mesh filename=franka_description/meshes/collision/link4.stl; visual mesh filename=franka_description/meshes/visual/link4.dae
- link panda_link5: geometry collision mesh filename=franka_description/meshes/collision/link5.stl; visual mesh filename=franka_description/meshes/visual/link5.dae
- link panda_link6: geometry collision mesh filename=franka_description/meshes/collision/link6.stl; visual mesh filename=franka_description/meshes/visual/link6.dae
- link panda_link7: geometry collision mesh filename=franka_description/meshes/collision/link7.stl; visual mesh filename=franka_description/meshes/visual/link7.dae
- link robotiq_2f_85_base: geometry collision mesh filename=robotiq-2f/meshes/collision/base.stl scale=0.001 0.001 0.001; visual mesh filename=robotiq-2f/meshes/visual/base.obj scale=0.1 0.1 0.1
- link robotiq_2f_85_left_coupler: geometry collision mesh filename=robotiq-2f/meshes/collision/coupler.stl scale=0.001 0.001 0.001; visual mesh filename=robotiq-2f/meshes/visual/coupler.obj scale=0.1 0.1 0.1
- link robotiq_2f_85_left_driver: geometry collision mesh filename=robotiq-2f/meshes/collision/driver.stl scale=0.001 0.001 0.001; visual mesh filename=robotiq-2f/meshes/visual/driver.obj scale=0.1 0.1 0.1
- link robotiq_2f_85_left_follower: geometry visual mesh filename=robotiq-2f/meshes/visual/follower.obj scale=0.1 0.1 0.1
- link robotiq_2f_85_left_pad: geometry collision mesh filename=robotiq-2f/meshes/collision/pad.stl scale=0.001 0.001 0.001; visual mesh filename=robotiq-2f/meshes/visual/pad.stl scale=0.0001 0.0001 0.0001
- link robotiq_2f_85_left_spring_link: geometry visual mesh filename=robotiq-2f/meshes/visual/spring_link.obj scale=0.1 0.1 0.1
- link robotiq_2f_85_right_coupler: geometry collision mesh filename=robotiq-2f/meshes/collision/coupler.stl scale=0.001 0.001 0.001; visual mesh filename=robotiq-2f/meshes/visual/coupler.obj scale=0.1 0.1 0.1
- link robotiq_2f_85_right_driver: geometry collision mesh filename=robotiq-2f/meshes/collision/driver.stl scale=0.001 0.001 0.001; visual mesh filename=robotiq-2f/meshes/visual/driver.obj scale=0.1 0.1 0.1
- link robotiq_2f_85_right_follower: geometry collision mesh filename=robotiq-2f/meshes/collision/follower.stl scale=0.001 0.001 0.001; visual mesh filename=robotiq-2f/meshes/visual/follower.obj scale=0.1 0.1 0.1
- link robotiq_2f_85_right_pad: geometry collision mesh filename=robotiq-2f/meshes/collision/pad.stl scale=0.001 0.001 0.001; visual mesh filename=robotiq-2f/meshes/visual/pad.stl scale=0.0001 0.0001 0.0001
- link robotiq_2f_85_right_spring_link: geometry collision mesh filename=robotiq-2f/meshes/collision/spring_link.stl scale=0.001 0.001 0.001; visual mesh filename=robotiq-2f/meshes/visual/spring_link.obj scale=0.1 0.1 0.1

Commit message: Created visual obj files from stl. Fixed visual mesh scaling.

File: mani_skill2_real2sim/assets/descriptions/panda_robotiq_85.urdf (robot description, URDF)
Before this commit: robot panda, 21 links, 20 joints
Links:
- link robotiq_2f_85_base: geometry collision mesh filename=robotiq-2f/meshes/collision/base.stl scale=0.001 0.001 0.001; visual mesh filename=robotiq-2f/meshes/visual/base.obj scale=0.001 0.001 0.001
- link robotiq_2f_85_left_coupler: geometry collision mesh filename=robotiq-2f/meshes/collision/coupler.stl scale=0.001 0.001 0.001; visual mesh filename=robotiq-2f/meshes/visual/coupler.obj scale=0.001 0.001 0.001
- link robotiq_2f_85_left_driver: geometry collision mesh filename=robotiq-2f/meshes/collision/driver.stl scale=0.001 0.001 0.001; visual mesh filename=robotiq-2f/meshes/visual/driver.obj scale=0.001 0.001 0.001
- link robotiq_2f_85_left_follower: geometry visual mesh filename=robotiq-2f/meshes/visual/follower.obj scale=0.001 0.001 0.001
- link robotiq_2f_85_left_pad: geometry collision mesh filename=robotiq-2f/meshes/collision/pad.stl scale=0.001 0.001 0.001; visual mesh filename=robotiq-2f/meshes/visual/pad.obj scale=0.001 0.001 0.001
- link robotiq_2f_85_left_spring_link: geometry visual mesh filename=robotiq-2f/meshes/visual/spring_link.obj scale=0.001 0.001 0.001
- link robotiq_2f_85_right_coupler: geometry collision mesh filename=robotiq-2f/meshes/collision/coupler.stl scale=0.001 0.001 0.001; visual mesh filename=robotiq-2f/meshes/visual/coupler.obj scale=0.001 0.001 0.001
- link robotiq_2f_85_right_driver: geometry collision mesh filename=robotiq-2f/meshes/collision/driver.stl scale=0.001 0.001 0.001; visual mesh filename=robotiq-2f/meshes/visual/driver.obj scale=0.001 0.001 0.001
- link robotiq_2f_85_right_follower: geometry collision mesh filename=robotiq-2f/meshes/collision/follower.stl scale=0.001 0.001 0.001; visual mesh filename=robotiq-2f/meshes/visual/follower.obj scale=0.001 0.001 0.001
- link robotiq_2f_85_right_pad: geometry collision mesh filename=robotiq-2f/meshes/collision/pad.stl scale=0.001 0.001 0.001; visual mesh filename=robotiq-2f/meshes/visual/pad.obj scale=0.001 0.001 0.001
- link robotiq_2f_85_right_spring_link: geometry collision mesh filename=robotiq-2f/meshes/collision/spring_link.stl scale=0.001 0.001 0.001; visual mesh filename=robotiq-2f/meshes/visual/spring_link.obj scale=0.001 0.001 0.001
